File: garage-console/hardware/garage-console.kicad_sch (KiCad schematic)
At the start: 39 parts, among them J1 XH-2P, J10 XH-2P, J11 XH-2P, J12 XH-2P, J13 XH-2P, J14 XH-2P, J15 XH-2P, J16 XH-2P, J2 XH-2P, J3 XH-2P, J4 XH-2P, J5 XH-2P, J6 XH-2P, J7 XH-2P, J8 XH-2P, J9 XH-2P, U1 XIAO-ESP32-C6, U2 PCF8575

Commit message: garage-console: drop U1 footprint, correct header spacing, exclude THT headers from assembly
The XIAO module now has no schematic symbol or PCB footprint at all;
its real connections are carried entirely by HDR1/HDR2 (two 1x7
2.54mm female sockets), with the module's own male pins plugging in
by hand off-board. This avoids the permanent DRC parity warning a
zero-pad placeholder footprint produced. HDR1/HDR2 spacing was
corrected to 15.24mm (from Seeed's authoritative OPL library, the
prior extraction had picked up a cosmetic pad on one side and an
averaged position on the other), and both are now excluded from the
JLCPCB assembly BOM/CPL so they can be hand-soldered instead of
fighting an unresolved placement-rotation convention mismatch in the
assembly toolchain.

Also: project-local symbol library for the two named-pin header
symbols, filter cap mirror-symmetry fixes, and .gitignore now excludes
fab_export/ and jlcpcb/ (regenerable fabrication/assembly artifacts,
not source) plus stray calibration project files.
Parts:
- removed U1: XIAO-ESP32-C6, Seeed_Studio_XIAO_Series:XIAO-ESP32-C6-DIP, symbol Seeed_Studio_XIAO_Series:XIAO-ESP32-C6-DIP
- added HDR1: Header_1x7_2.54mm, Connector_PinSocket_2.54mm:PinSocket_1x07_P2.54mm_Vertical, symbol garage_console:XIAO_HDR_A
- added HDR2: Header_1x7_2.54mm, Connector_PinSocket_2.54mm:PinSocket_1x07_P2.54mm_Vertical, symbol garage_console:XIAO_HDR_B
Connections:
- net +3V3: now also HDR2.5 (+3V3)
- net GND: now also HDR2.6 (GND)
- net PCF_INT: now also HDR1.3 (PCF_INT)
- net SCL: now also HDR1.6 (SCL)
- net SDA: now also HDR1.5 (SDA)
- no-connect marks 9 -> 23
