File: garage-console/hardware/garage-console.kicad_sch (KiCad schematic)
At the start: 40 parts, among them J1 XH-2P, J10 XH-2P, J11 XH-2P, J12 XH-2P, J13 XH-2P, J14 XH-2P, J15 XH-2P, J16 XH-2P, J2 XH-2P, J3 XH-2P, J4 XH-2P, J5 XH-2P, J6 XH-2P, J7 XH-2P, J8 XH-2P, J9 XH-2P, U2 PCF8575

Commit message: garage-console: assemble the headers, rename U2 to U1, add CPL corrections
Headers are populated by the fab after all — JLCPCB's Economic tier does
support through-hole (single-sided SMT/thru-hole placement), so HDR1/HDR2
no longer need to be held back for hand-soldering. Cleared their
exclude_from_bom/exclude_from_pos_files flags and set in_bom yes on both
symbols; they're back in the BOM and the CPL is 40 rows.

U2 -> U1: the PCF8575 is the only IC on the board, and U1 was freed when
the XIAO module's footprint was dropped. Renamed across schematic, PCB and
README; DRC schematic parity stayed at 0, so the symbol/footprint link
survived.

jlcpcb-cpl-corrections.json records the placement corrections verified in
JLCPCB's Component Placements preview, so regenerating the fab package
doesn't silently lose them:

- rotation: JST XH +180, SSOP-24 +90, 1x7 sockets +90
- position: JST +1.25mm X, HDR1 +7.62mm Y, HDR2 -7.62mm Y

The position offsets work around Konnect issue #667 — CPL Mid X/Mid Y
carries the KiCad footprint anchor instead of the component midpoint, so
anything anchored on pin 1 lands off by the anchor-to-centre vector. U1
needs no offset because the SSOP-24 anchor is already centred, which is
why that one always looked right. Remove the offsets if #667 is fixed, or
they will double-correct; the policy's provenance field says so too.

Co-Authored-By: Claude Opus 5 (1M context) <noreply@anthropic.com>
Parts:
- HDR1, HDR2: now in the parts list
- renumbered U2 to U1
Changed lines of the file:
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@@
 		(on_board yes)
 		(dnp no)
-		(property "Reference" "U2"
+		(property "Reference" "U1"
 			(at 173.99 105.41 0)
 			(effects
@@
 			(project "garage-console"
 				(path "931ac6af-e45c-4c9e-b8b9-f003eb1d1d30"
-					(reference "U2")
+					(reference "U1")
 					(unit 1)
 				)
@@
 		(at 76.2 139.7 0)
 		(unit 1)
-		(in_bom no)
+		(in_bom yes)
 		(on_board yes)
 		(dnp no)
@@
 		(at 76.2 180.34 0)
 		(unit 1)
-		(in_bom no)
-		(on_board yes)
-		(dnp no)
+		(in_bom yes)
+		(on_board yes)
+		(dnp no)
