File: garage-water-tank/hardware/garage-water-tank.kicad_sch (KiCad schematic)
At the start: 10 parts, among them J1 Conn_01x04, J2 Conn_01x04, SW1 SW_Push

Commit message: garage-water-tank: regenerate fab files, add CPL corrections, fix R2's library
Generates the upload-ready JLCPCB package (gerbers, drill, BOM, CPL) for
the socketed layout, tracked the way garage-console tracks its own.

Adds jlcpcb-cpl-corrections.json. HDR1/HDR2 need the same pin-1-anchor
compensation garage-console documented: Konnect writes the footprint
anchor into CPL Mid X/Mid Y rather than the component midpoint
(Konnect #667), so the 1x7 sockets land 7.62mm out in opposite board-Y
directions. With the offsets applied both headers land on y=-67.6815,
the line they physically share. J2 needs +3.0mm in X for the same
reason (JST PH pads at local x 0/2/4/6). The 90 deg socket rotation is
carried over from garage-console, where this exact footprint was
verified in JLCPCB's placement preview; J1 and J2 rotations are NOT yet
verified and are called out as such in the policy's provenance.

Fixes R2, which pointed at "Resistor_SMD_test:R_0805_2012Metric" -- a
nickname that resolves in no library table and matches no .pretty on
disk. Its geometry is identical to R1/R3/R4's stock
Resistor_SMD:R_0805_2012Metric, and the dangling nickname was splitting
two identical 4k7 0805s across separate BOM lines. Every footprint
nickname on the board now resolves.

SW1 is correctly absent from both BOM and CPL.

Not ready to order: validate_for_manufacturing returns NOT READY on the
two pre-existing J1 copper-edge-clearance errors (its own Edge.Cuts
circles sit 0.1mm from its pads against a 0.5mm rule), and every part
except J2 still lacks an LCSC number.

Co-Authored-By: Claude Opus 5 (1M context) <noreply@anthropic.com>
Parts:
- R2: footprint Resistor_SMD_test:R_0805_2012Metric -> Resistor_SMD:R_0805_2012Metric
Changed lines of the file:
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@@
 			)
 		)
-		(property "Footprint" "Resistor_SMD_test:R_0805_2012Metric"
+		(property "Footprint" "Resistor_SMD:R_0805_2012Metric"
 			(at 173.482 93.98 90)
 			(hide yes)

Commit message: garage-water-tank: source LCSC parts for the whole BOM, fix J2's connector
Every BOM line now carries an LCSC number, so the board can be quoted
for assembly. SW1 stays out — it is hand-soldered from spares.

Reused from garage-console, all verified in stock against the JLCPCB
parts database: C49678 (100nF 0805 X7R, Basic), C17673 (4.7k 0805,
Basic), C22438157 (hanxia HX PM2.54-1x7P ZC-Y, the 8.5mm socket the
header approach depends on).

Sourced new: C17408 for R3/R4 — 100R 0805 1%, Basic library, the same
UNI-ROYAL 0805W8F series garage-console's resistors come from. And
C42379197 for J1, an SMD staggered-pin 1x4 2.54mm socket matching the
footprint's pad pattern; 5mm body, chosen for "low profile" as the
footprint and 3D model names both say. Worth confirming that height
suits the OLED stack before ordering.

Fixes J2, which carried LCSC C144395 and MPN "B4B-XH-A" — a JST XH at
2.5mm pitch — against a footprint drilled for JST PH at 2.00mm. That
part cannot physically fit the holes. Replaced with C131334
(B4B-PH-K-S), PH 2mm, 4-pin, through hole, 211k in stock. The
footprint was always the deliberate choice: the A02YYUW sensor ships a
PH cable, and the datasheets are in hardware/datasheets.

Footprint fields are synced with the symbols, so schematic parity stays
at zero; adding LCSC to the symbols alone had opened 8 parity warnings.

Co-Authored-By: Claude Opus 5 (1M context) <noreply@anthropic.com>
Parts:
- C1: LCSC (none) -> C49678
- HDR1, HDR2: LCSC (none) -> C22438157
- J1: LCSC (none) -> C42379197; MPN https://www.aliexpress.com/item/1005006410708666.html -> HX PM2.54-1x4P TP-YQ; Manufacturer (none) -> hanxia
- J2: LCSC C144395 -> C131334; MPN B4B-XH-A -> B4B-PH-K-S(LF)(SN)
- R1, R2: LCSC (none) -> C17673
- R3, R4: LCSC (none) -> C17408
Changed lines of the file:
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@@
 			)
 		)
-	)
+		(property "LCSC" "C49678"
+			(at 180.34 130.81 0)
+			(hide yes)
+			(effects
+				(font
+					(size 1.27 1.27)
+				)
+			)
+		))
 	(symbol
 		(lib_id "Device:R_Small")
@@
 			)
 		)
-	)
+		(property "LCSC" "C17408"
+			(at 180.34 138.43 0)
+			(hide yes)
+			(effects
+				(font
+					(size 1.27 1.27)
+				)
+			)
+		))
 	(symbol
 		(lib_id "Device:R_Small")
@@
 			)
 		)
-	)
+		(property "LCSC" "C17408"
+			(at 180.34 135.89 0)
+			(hide yes)
+			(effects
+				(font
+					(size 1.27 1.27)
+				)
+			)
+		))
 	(symbol
 		(lib_id "Device:R")
@@
 			)
 		)
-	)
+		(property "LCSC" "C17673"
+			(at 175.26 93.98 0)
+			(hide yes)
+			(effects
+				(font
+					(size 1.27 1.27)
+				)
+			)
+		))
 	(symbol
 		(lib_id "Connector_Generic:Conn_01x04")
@@
 			)
 		)
-		(property "MPN" "B4B-XH-A"
+		(property "MPN" "B4B-PH-K-S(LF)(SN)"
 			(at 193.04 133.35 0)
 			(hide yes)
@@
 			)
 		)
-		(property "LCSC" "C144395"
+		(property "LCSC" "C131334"
 			(at 193.04 127.635 0)
 			(hide yes)
@@
 			)
 		)
-	)
+		(property "LCSC" "C17673"
+			(at 171.45 93.98 0)
+			(hide yes)
+			(effects
+				(font
+					(size 1.27 1.27)
+				)
+			)
+		))
 	(symbol
 		(lib_id "power:VCC")
@@
 			)
 		)
-		(property "MPN" "https://www.aliexpress.com/item/1005006410708666.html"
+		(property "MPN" "HX PM2.54-1x4P TP-YQ"
 			(at 181.61 104.14 0)
 			(hide yes)
@@
 			)
 		)
-		(property "Manufacturer" ""
+		(property "Manufacturer" "hanxia"
 			(at 181.61 104.14 0)
 			(hide yes)
@@
 			)
 		)
-	)
+		(property "LCSC" "C42379197"
+			(at 181.61 104.14 0)
+			(hide yes)
+			(effects
+				(font
+					(size 1.27 1.27)
+				)
+			)
+		))
 	(symbol
 		(lib_id "garage_water_tank:XIAO_HDR_A")
@@
 			)
 		)
-	)
+		(property "LCSC" "C22438157"
+			(at 104.14 106.68 0)
+			(hide yes)
+			(effects
+				(font
+					(size 1.27 1.27)
+				)
+			)
+		))
 	(symbol
 		(lib_id "garage_water_tank:XIAO_HDR_B")
@@
 			)
 		)
-	)
+		(property "LCSC" "C22438157"
+			(at 101.6 130.81 0)
+			(hide yes)
+			(effects
+				(font
+					(size 1.27 1.27)
+				)
+			)
+		))
 	(symbol
 		(lib_id "power:PWR_FLAG")
