File: garage-water-tank/hardware/garage-water-tank.kicad_pcb (KiCad board)
At the start: 2 copper layers, 35.3 x 39.4 mm, 10 parts, among them J1 Conn_01x04, J2 Conn_01x04, SW1 SW_Push

Commit message: garage-water-tank: silkscreen the XIAO's USB-C overhang and label it
Marks where the module's USB-C connector sits, which is otherwise
invisible on the bare board: the module has no footprint here, so
nothing on the PCB showed the port's outline or which end it faces.
Useful when cutting the enclosure opening.

Geometry is lifted from Seeed's own OPL footprint
(Seeed Studio XIAO Series Library/XIAO-ESP32-C6-DIP), taking only the
silkscreen beyond the module body — its F.Fab/courtyard rect ends at
local x 10.55, so the three lines and two r=0.5 corner arcs past that
are the connector overhang and nothing else. Transformed by the
placement the deleted U1 footprint had, origin (139.7, 67.6815) at
-90 deg, so local (lx,ly) maps to (139.7 - ly, 67.6815 + lx).

Result checks out against the module: 9.00mm wide, centred on x = 139.7
which is the midline between the two header columns, protruding 1.51mm
past the module edge at y = 78.2225. The 3D render puts the USB-C model
exactly over it.

A "USB" label goes below at (139.7, 81.3), clear of the module body so
it stays readable with the board assembled, at 1mm height and 0.15mm
thickness to satisfy the project's silkscreen rule.

DRC unchanged: 0 errors, no new silk violations. Regenerated fab shows
F_Silkscreen.gto as the only altered file, every other layer and both
drill files byte-identical.

Co-Authored-By: Claude Opus 5 (1M context) <noreply@anthropic.com>
Other:
- board text added: "USB"
Changed lines of the file:
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@@
+	)
+	(gr_line
+		(start 135.196 79.2325)
+		(end 135.196 78.2225)
+		(stroke
+			(width 0.127)
+			(type default)
+		)
+		(layer "F.SilkS")
+	)
+	(gr_arc
+		(start 135.696 79.7325)
+		(mid 135.342447 79.586053)
+		(end 135.196 79.2325)
+		(stroke
+			(width 0.127)
+			(type default)
+		)
+		(layer "F.SilkS")
+	)
+	(gr_line
+		(start 143.6913 79.7325)
+		(end 135.696 79.7325)
+		(stroke
+			(width 0.127)
+			(type default)
+		)
+		(layer "F.SilkS")
+	)
+	(gr_arc
+		(start 144.1913 79.2328)
+		(mid 144.044747 79.58616)
+		(end 143.6913 79.7325)
+		(stroke
+			(width 0.127)
+			(type default)
+		)
+		(layer "F.SilkS")
+	)
+	(gr_line
+		(start 144.195 78.2225)
+		(end 144.1913 79.2328)
+		(stroke
+			(width 0.127)
+			(type default)
+		)
+		(layer "F.SilkS")
 	)
 	(gr_line
@@
 		(layer "Edge.Cuts")
 	)
+	(gr_text "USB"
+		(at 139.7 81.3 0)
+		(layer "F.SilkS")
+		(effects
+			(font
+				(size 1 1)
+				(thickness 0.15)
+			)
+		)
+	)
 	(gr_text "garage-\nwater-tank\nv02"

Commit message: garage-water-tank: mirror J1's pad stagger for the YQ socket, shift 0.355mm off the edge
Option B of the J1 variant problem. JLCPCB's placement preview showed
every one of J1's four SMD legs landing on the opposite side from its
pad. That cannot be fixed by rotation: for a 4-position alternating
stagger, 180 deg maps pins 1234 to positions 4321 and flips each side,
so the left-to-right side pattern comes back identical. Only the part
variant or the footprint can change it.

Seeed's supplier ships both: the ordered C42379197 is HX PM2.54-1x4P
TP-YQ, boxed as B-type "right front", while C48641754 is the ZQ
"left front" mirror. ZQ exists only at 8.5mm body height though, and
the module height matters here because the OLED's legs pass through the
board and set its standoff. So the footprint is mirrored instead,
keeping the 5mm part: each copper pad's local X is negated, the NPTH
leg bores sit on the axis at x=0 and do not move.

Mirroring put VCC and SDA on the row nearest the board edge, where DRC
then objected at 0.145mm against a 0.5mm rule. That margin was always
out of spec — it just sat on GND and SCL before — so J1 moves up
0.355mm (origin y 93.375 -> 93.020), landing the clearance on exactly
0.500mm. KiCad measures in integer nanometres, so exactly-equal passes;
the check confirms it. This is the first time that pre-existing
marginality has actually been in spec.

Knock-on work, all verified:
- SCL, VCC and SDA re-routed to the swapped pad sides, weaving between
  the Ø1.0mm leg holes with >= 1.0mm to each hole centre
- J1's silkscreen rebuilt from the library so its gaps line up with the
  pads again; the board instance had silently kept the old geometry
  because SetStart/SetEnd on a footprint's child shapes do not update
  the stored local coordinates
- re-routing pinched the F.Cu GND pour into two islands and orphaned
  the second; a GND stitching via at (140.75, 69.00), the clearest
  point in that island at 2.10mm, ties it through the B.Cu pour

DRC: 0 err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
Parts:
- moved J1 0.36 mm to (140.0, 93.0)
Routing:
- net SDA: track 30.0 -> 35.1 mm
- net VCC: track 48.2 -> 52.5 mm
- net SCL: track 37.1 -> 33.8 mm
- net GND: vias 0 -> 1
