File: garage-water-tank/hardware/garage-water-tank.kicad_pcb (KiCad board)
At the start: 2 copper layers, 35.3 x 39.4 mm, 10 parts, among them J1 Conn_01x04, J2 Conn_01x04, SW1 SW_Push

Commit message: garage-water-tank: owner's placement pass, repair the VCC break it left
Manual rework by the project owner: C1, R3 and R4 repositioned and
rotated, R2 nudged 0.5mm. Routing improves again — 53 segments to 40,
200.82mm to 187.52mm, and the via count drops 3 to 1 by removing the
TX and J2-Pin_4 vias, so those nets are now single-layer. The GND
stitching via was kept and moved to (140.5, 71.5), still doing its job
of tying the second F.Cu pour island through B.Cu.

Moving R2 from y=65.5 to 65.0 truncated the trace that used to carry
VCC on up to R1, leaving R1 pad 1 orphaned — DRC caught it as a missing
connection between the two 4k7 pull-ups. Repaired with a straight F.Cu
segment from (142.0875, 65.0) to (142.0875, 62.5); the corridor was
measured clear first, nearest foreign copper 0.912mm against the
0.45mm needed.

Checks: ERC 0, DRC 0 errors, 0 unconnected, 0 schematic parity, all 9
CPL rows on their measured pad centres. The invariants hold — J1 still
exactly 0.5000mm off the board edge, SW1 untouched on B.Cu.

J1's lib_footprint_mismatch is back and will keep coming back: KiCad's
own save re-serialises stroke style as "default" and the NPTH pad
rotation absolutely, which is what d219d6c had normalised by script.
The library copy, written through the scripting API, is the one using
"solid". Not worth fighting per-save; the geometry is identical.

Co-Authored-By: Claude Opus 5 (1M context) <noreply@anthropic.com>
Parts:
- moved R4 8.06 mm to (143.0, 60.0), turned to 180 degrees
- moved C1 2.04 mm to (135.5, 69.2), turned to 90 degrees
- moved R3 0.56 mm to (135.5, 60.8), turned to -90 degrees
- moved R2 0.50 mm to (143.0, 65.0)
Routing:
- net TX: track 13.9 -> 3.43 mm, vias 1 -> 0
- net Net-(J2-Pin_4): track 16.2 -> 20.0 mm, vias 1 -> 0
- net VCC: track 52.5 -> 50.1 mm
- net Net-(J2-Pin_3): track 14.0 -> 12.0 mm
